File: Hardware/PCB/Eagle/Jacdac_Pressure_Sensor.brd (EAGLE design)
At the start: 33.8 x 27.9 mm, 30 parts, among them J1 JACDAC-CONNECTOR, J2 SWD-ADAPTER-, J3 HEADER_MALE-1X07, U1 NCP114ASN330T1G, U2 STM32F042F6P6, U3 BAT54S,235, U4 LPS33HWTR

Commit message: Updated PCB files
Parts:
- removed LABEL1: MMC-LOGO-SM, MMC Eagle:MMC_SMALL_LOGO
- added C5: 33pF, milador_SMD:0603
- C1, C4: value 33pF -> 1uF; device milador_SMD:0603 -> milador_SMD:0603-NO
- C2: value 1uF -> 33pF; device milador_SMD:0603-NO -> milador_SMD:0603
- C3: value 1uF -> 0.1uF
- SJ1, SJ2: device milador_SMD:SOLDERJUMPER_OPENED_TRACE_SILK -> milador_SMD:SOLDERJUMPER_CLOSEDWIRE
- moved C3 20.0 mm to (7.62, 21.1), turned to 180 degrees
- moved C4 10.9 mm to (15.2, 2.54)
- moved C1 2.54 mm to (9.14, 13.5)
- moved C2 2.54 mm to (9.14, 16.0)
- moved R5 2.54 mm to (20.3, 13.5)
- moved R6 2.54 mm to (20.3, 16.0)
- moved U$1 0.25 mm to (17.0, 13.5)
- moved U$2 0.25 mm to (17.0, 16.3)
Connections:
- net +3V3: now also C5.1
- net GND: now also C5.2
- net N$4: now also C2.1; no longer C1.1
- net N$6: now also R6.1; no longer R5.1
- net N$7: now also R5.1; no longer R6.1
- net VCC: now also C1.1; no longer C2.1
Routing:
- net +3V3: track 75.9 -> 80.4 mm
