File: Hardware/PCB/Eagle/Jacdac_Pressure_Sensor_Maker.brd (EAGLE design)
At the start: 33.8 x 27.9 mm, 30 parts, among them J1 JACDAC-CONNECTOR, J2 SWD-ADAPTER-, J3 HEADER_MALE-1X07, U1 NCP114ASN330T1G, U2 STM32F042F6P6, U3 BAT54S,235, U4 LPS33HWTR

Commit message: Updated PCB files
Parts:
- removed LABEL1: MMC-LOGO-SM, MMC Eagle:MMC_SMALL_LOGO
- added C5: 33pF, milador_SMD:0805-MP
- C1, C4: value 33pF -> 1uF; device milador_SMD:0603 -> milador_SMD:0805-MP
- C2: value 1uF -> 33pF; device milador_SMD:0603-NO -> milador_SMD:0805-MP
- C3: value 1uF -> 0.1uF; device milador_SMD:0603-NO -> milador_SMD:0805-MP
- D2, D3: value STS521050BL90 -> RCLAMP0521PATCT
- R1, R2, R3, R4, R5, R6: device milador_SMD:0603 -> milador_SMD:0805-MP
- SJ1, SJ2: device milador_SMD:SOLDERJUMPER_OPENED_TRACE_SILK -> milador_SMD:SOLDERJUMPER_CLOSEDWIRE
- moved C3 20.0 mm to (7.62, 21.1), turned to 180 degrees
- moved C4 10.9 mm to (15.2, 2.54)
- moved C1 2.54 mm to (9.14, 13.5)
- moved C2 2.54 mm to (9.14, 16.0)
- moved R5 2.54 mm to (20.3, 13.5)
- moved R6 2.54 mm to (20.3, 16.0)
- moved U1 0.25 mm to (3.81, 8.89)
- moved U$1 0.25 mm to (17.0, 13.5)
- moved U$2 0.25 mm to (17.0, 16.3)
Connections:
- net +3V3: now also C5.1
- net GND: now also C5.2, D2.1, D3.1; no longer D2.A, D3.A
- net N$17: now also D3.2; no longer D3.K
- net N$4: now also C2.1; no longer C1.1
- net N$6: now also R6.1; no longer R5.1
- net N$7: now also R5.1; no longer R6.1
- net VCC: now also C1.1, D2.2; no longer C2.1, D2.K
Routing:
- net +3V3: track 75.9 -> 80.6 mm
- net N$7: track 5.98 -> 6.48 mm
