File: Hardware/PCB/Eagle/Jacdac_Pressure_Sensor_Maker.brd (EAGLE design)
At the start: 33.8 x 27.9 mm, 30 parts, among them J1 JACDAC-CONNECTOR, J2 SWD-ADAPTER-, J3 HEADER_MALE-1X07, U1 NCP114ASN330T1G, U2 STM32F042F6P6, U3 BAT54S,235, U4 LPS33HWTR

Commit message: Updated design
Use I2C instead of SPI
Parts:
- added U$3: MMC-LOGO-SM, MMC Eagle:MMC_SMALL_LOGO
- J1: value JACDAC-CONNECTOR -> JACDAC_EDGE_CONN-INNIE; device milador:JACDAC-CONNECTOR -> Jacdac:JACDAC-EDGE-CONN-INNIE
Connections:
- removed net N$17: D3.2, FB1.2, J1.P3
- removed net SCK: J3.3, SJ1.1, U2.11, U4.2
- new net J_DATA: D3.2, FB1.2, J1.JD1, J1.JD2, J1.JD3
- new net SCL: J3.3, SJ1.1, U2.17, U4.2
- net GND: now also J1.GND1, J1.GND2, J1.GND3, J1.GND4; no longer J1.P2
- net SDA: now also U2.18; no longer U2.13
- net VCC: now also J1.VDD1, J1.VDD2, J1.VDD3; no longer J1.P1
Routing:
- net SCK: track 34.9 -> 0.00 mm, vias 2 -> 0
- net SCL: track 0.00 -> 30.2 mm, vias 0 -> 2
- net J_DATA: track 0.00 -> 19.8 mm
- net N$17: track 10.3 -> 0.00 mm
- net VCC: track 17.0 -> 23.7 mm
- net SDA: track 33.3 -> 29.3 mm
- net GND: track 14.7 -> 16.4 mm
- net RESET: track 13.1 -> 12.4 mm
Other:
- board size 33.8 x 27.9 mm -> 27.9 x 27.9 mm
- board text added: "SCL"
- board text removed: "SCK"
