File: Hardware/PCB/Eagle/Jacdac_Pressure_Sensor.sch (EAGLE design)
At the start: 30 parts, among them J1 JACDAC-CONNECTOR, J2 SWD-ADAPTER-, J3 HEADER_MALE-1X07, U1 NCP114ASN330T1G, U2 STM32F042F6P6, U3 BAT54S,235, U4 LPS33HWTR

Commit message: Updated PCB files
Parts:
- removed LABEL1: MMC-LOGO-SM, MMC Eagle:MMC-LOGO-SM
- added C5: 33pF, milador_SMD:CAP_CERAMIC-0603
- C1, C4: value 33pF -> 1uF; device milador_SMD:CAP_CERAMIC-0603 -> milador_SMD:CAP_CERAMIC-0603-NO
- C2: value 1uF -> 33pF; device milador_SMD:CAP_CERAMIC-0603-NO -> milador_SMD:CAP_CERAMIC-0603
- C3: value 1uF -> 0.1uF
- D2, D3: device milador_SMD:RCLAMP0521PATCT -> milador_SMD:DIODE-ZENER-AA-RCLAMP0521PATCT
- SJ1, SJ2: device milador_SMD:SOLDERJUMPEROPENED -> milador_SMD:SOLDERJUMPERCLOSED
Connections:
- net +3V3: now also C5.1
- net GND: now also C5.2
- net N$17: now also D3.A2; no longer D3.C
- net N$4: now also C2.1; no longer C1.1
- net N$6: now also R6.1; no longer R5.1
- net N$7: now also R5.1; no longer R6.1
- net VCC: now also C1.1, D2.A2; no longer C2.1, D2.C
Other:
- moved on the sheet: C1, C2, C3, C4, R5, R6

Commit message: Updated design
Use I2C instead of SPI
Parts:
- J1: value JACDAC-CONNECTOR -> JACDAC_EDGE_CONN-INNIE; device milador:JACDAC-CONNECTOR -> Jacdac:JACDAC_EDGE_CONN-INNIE
Connections:
- removed net N$17: D3.A2, FB1.2, J1.JDF
- removed net SCK: J3.3, SJ1.1, U2.PA5, U4.SCL/SPC
- new net J_DATA: D3.A2, FB1.2, J1.1
- new net SCL: J3.3, SJ1.1, U2.PA11, U4.SCL/SPC
- net GND: now also J1.2; no longer J1.GND
- net SDA: now also U2.PA12; no longer U2.PA7
- net VCC: now also J1.3; no longer J1.JD5V

Commit message: Corrected Capacitor values
Parts:
- C5: value 33pF -> 1uF
Changed lines of the file:
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@@
 <part name="FRAME1" library="frames" library_urn="urn:adsk.eagle:library:229" deviceset="A3L-LOC" device=""/>
 <part name="+3V5" library="supply1" library_urn="urn:adsk.eagle:library:371" deviceset="+3V3" device=""/>
-<part name="C5" library="milador_SMD" library_urn="urn:adsk.eagle:library:27847482" deviceset="CAP_CERAMIC-" device="0603" package3d_urn="urn:adsk.eagle:package:29222124/2" value="33pF"/>
+<part name="C5" library="milador_SMD" library_urn="urn:adsk.eagle:library:27847482" deviceset="CAP_CERAMIC-" device="0603" package3d_urn="urn:adsk.eagle:package:29222124/2" value="1uF"/>
 <part name="GND9" library="SparkFun-PowerSymbols" deviceset="GND" device=""/>
 <part name="GND10" library="SparkFun-PowerSymbols" deviceset="GND" device=""/>

Commit message: Updated main design
Centering the sensor
Parts:
- removed J3: HEADER_MALE-1X07, milador:HEADER_MALE-1X07
- removed SJ1, SJ2: (no value), milador_SMD:SOLDERJUMPERCLOSED
- removed U$1: MILADOR-PIN-NAME-SDA, milador:MILADOR-PIN-NAME-SDA
- removed U$2: MILADOR-PIN-NAME-SCK, milador:MILADOR-PIN-NAME-SCK
- added H1, H3: MOUNTINGHOLE3.0THIN, milador:MOUNTINGHOLE3.0THIN
- C1: value 1uF -> 0.1uF
- C2: value 33pF -> 1uF; device milador_SMD:CAP_CERAMIC-0603 -> milador_SMD:CAP_CERAMIC-0603-NO
- C3: value 0.1uF -> 33pF; device milador_SMD:CAP_CERAMIC-0603-NO -> milador_SMD:CAP_CERAMIC-0603
- H2, JP3: value STAND-OFF-3.0 -> MOUNTINGHOLE3.0THIN; device milador:STAND-OFF-3.0 -> milador:MOUNTINGHOLE3.0THIN
- U3: value BAT54S,235 -> LPS33HWTR; device milador_SMD:BAT54S,235 -> milador_SMD:LPS33HWTR
- U4: value LPS33HWTR -> BAT54S,235; device milador_SMD:LPS33HWTR -> milador_SMD:BAT54S,235
Connections:
- removed net CS: J3.6, U4.CS
- removed net INT: J3.7, U4.INT_DRDY
- removed net N$6: R6.1, SJ1.2
- removed net N$7: R5.1, SJ2.2
- removed net SDO: J3.5, U4.SDO/SA0
- net +3V3: now also C1.1, U3.VDD, U3.VDD_IO, U4.S; no longer C3.1, J3.1, U3.S, U4.VDD, U4.VDD_IO
- net GND: now also U3.EXP_GND, U3.GND, U3.RES, U4.G; no longer J3.2, U3.G, U4.EXP_GND, U4.GND, U4.RES
- net JD_DATA: now also U4.D; no longer U3.D
- net N$4: now also C3.1; no longer C2.1
- net SCL: now also R5.1, U3.SCL/SPC; no longer J3.3, SJ1.1, U4.SCL/SPC
- net SDA: now also R6.1, U3.SDA/SDI/SDO; no longer J3.4, SJ2.1, U4.SDA/SDI/SDO
- net VCC: now also C2.1; no longer C1.1
Other:
- note removed: "Headers"
- moved on the sheet: C1, C2, C3, R5, R6

Commit message: Updated PCB
Parts:
- removed JP3: MOUNTINGHOLE3.0THIN, milador:MOUNTINGHOLE3.0THIN
- added H4: MOUNTINGHOLE2.5, milador:MOUNTINGHOLE2.5
- added MMC_LOGO: MMC_LOGO-SM, MMC Eagle:MMC_LOGO-SM
- added U$1: JACDAC-DEVICE-LPS33HW, milador:JACDAC-DEVICE-LPS33HW
- H1, H2, H3: value MOUNTINGHOLE3.0THIN -> MOUNTINGHOLE2.5; device milador:MOUNTINGHOLE3.0THIN -> milador:MOUNTINGHOLE2.5
Connections:
- net GND: now also H3.P$1, H4.P$1
- net J_DATA: now also H2.P$1
- net VCC: now also H1.P$1
Other:
- moved on the sheet: R5, R6, U3

Commit message: Updated design : Centered Pressure Sensor
Parts:
- D2, D3: device milador_SMD:DIODE-ZENER-AA-RCLAMP0521PATCT -> milador_SMD:DIODE-ZENER-RCLAMP0521PATCT
Connections:
- net +3V3: no longer U1.GND
- net GND: now also U1.GND
Other:
- moved on the sheet: C4
Changed lines of the file:
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@@
 <part name="+3V6" library="supply1" library_urn="urn:adsk.eagle:library:371" deviceset="+3V3" device=""/>
 <part name="GND11" library="SparkFun-PowerSymbols" deviceset="GND" device=""/>
-<part name="LABEL3" library="milador" library_urn="urn:adsk.eagle:library:12595918" deviceset="MILADOR-LOGO-" device="" package3d_urn="urn:adsk.eagle:package:28431737/1"/>
+<part name="LABEL3" library="milador" library_urn="urn:adsk.eagle:library:12595918" deviceset="MILADOR-LOGO-" device="" package3d_urn="urn:adsk.eagle:package:28431737/2"/>
 <part name="LABEL2" library="milador" library_urn="urn:adsk.eagle:library:12595918" deviceset="JACDAC-DEVICE-" device="PS" package3d_urn="urn:adsk.eagle:package:30748291/2"/>
 <part name="R5" library="milador_SMD" library_urn="urn:adsk.eagle:library:27847482" deviceset="RESISTOR-" device="0603" package3d_urn="urn:adsk.eagle:package:29222124/2" value="4.7K"/>
@@
 <part name="C1" library="milador_SMD" library_urn="urn:adsk.eagle:library:27847482" deviceset="CAP_CERAMIC-" device="0603-NO" package3d_urn="urn:adsk.eagle:package:27847599/2" value="0.1uF"/>
 <part name="GND2" library="SparkFun-PowerSymbols" deviceset="GND" device=""/>
-<part name="D2" library="milador_SMD" library_urn="urn:adsk.eagle:library:27847482" deviceset="DIODE-ZENER-AA-" device="RCLAMP0521PATCT" package3d_urn="urn:adsk.eagle:package:30689290/6" value="RCLAMP0521PATCT"/>
-<part name="D3" library="milador_SMD" library_urn="urn:adsk.eagle:library:27847482" deviceset="DIODE-ZENER-AA-" device="RCLAMP0521PATCT" package3d_urn="urn:adsk.eagle:package:30689290/6" value="RCLAMP0521PATCT"/>
+<part name="D2" library="milador_SMD" library_urn="urn:adsk.eagle:library:27847482" deviceset="DIODE-ZENER-" device="RCLAMP0521PATCT" package3d_urn="urn:adsk.eagle:package:30689290/6" value="RCLAMP0521PATCT"/>
+<part name="D3" library="milador_SMD" library_urn="urn:adsk.eagle:library:27847482" deviceset="DIODE-ZENER-" device="RCLAMP0521PATCT" package3d_urn="urn:adsk.eagle:package:30689290/6" value="RCLAMP0521PATCT"/>
 <part name="J1" library="Jacdac" library_urn="urn:adsk.eagle:library:30688326" deviceset="JACDAC_EDGE_CONN" device="-INNIE" package3d_urn="urn:adsk.eagle:package:30688335/1"/>
 <part name="H3" library="milador" library_urn="urn:adsk.eagle:library:12595918" deviceset="MOUNTINGHOLE" device="2.5" package3d_urn="urn:adsk.eagle:package:29232281/2" value="MOUNTINGHOLE2.5"/>
@@
 <attribute name="VALUE" x="73.66" y="192.786" size="1.778" layer="96" font="vector" align="top-center"/>
 </instance>
-<instance part="C4" gate="G$1" x="73.66" y="200.66" smashed="yes">
-<attribute name="NAME" x="71.37" y="201.91" size="1.27" layer="95" font="vector" rot="R90" align="center"/>
-<attribute name="VALUE" x="75.96" y="201.91" size="1.27" layer="96" font="vector" rot="R90" align="center"/>
+<instance part="C4" gate="G$1" x="73.66" y="208.534" smashed="yes">
+<attribute name="NAME" x="71.37" y="209.784" size="1.27" layer="95" font="vector" rot="R90" align="center"/>
+<attribute name="VALUE" x="75.96" y="209.784" size="1.27" layer="96" font="vector" rot="R90" align="center"/>
 </instance>
 <instance part="+3V1" gate="G$1" x="86.36" y="228.6" smashed="yes">
@@
 <pinref part="C4" gate="G$1" pin="2"/>
 <pinref part="GND3" gate="1" pin="GND"/>
-<wire x1="73.66" y1="198.12" x2="73.66" y2="195.58" width="0.1524" layer="91"/>
+<wire x1="73.66" y1="205.994" x2="73.66" y2="197.358" width="0.1524" layer="91"/>
+<wire x1="73.66" y1="197.358" x2="73.66" y2="195.58" width="0.1524" layer="91"/>
+<wire x1="30.48" y1="220.98" x2="30.48" y2="197.358" width="0.1524" layer="91"/>
+<pinref part="U1" gate="A" pin="GND"/>
+<wire x1="35.56" y1="220.98" x2="30.48" y2="220.98" width="0.1524" layer="91"/>
+<wire x1="30.48" y1="197.358" x2="73.66" y2="197.358" width="0.1524" layer="91"/>
+<junction x="73.66" y="197.358"/>
 </segment>
 <segment>
@@
 <net name="+3V3" class="0">
 <segment>
-<pinref part="U1" gate="A" pin="GND"/>
-<wire x1="35.56" y1="220.98" x2="30.48" y2="220.98" width="0.1524" layer="91"/>
-<wire x1="30.48" y1="220.98" x2="30.48" y2="208.28" width="0.1524" layer="91"/>
 <pinref part="C4" gate="G$1" pin="1"/>
-<wire x1="30.48" y1="208.28" x2="73.66" y2="208.28" width="0.1524" layer="91"/>
-<wire x1="73.66" y1="208.28" x2="73.66" y2="205.74" width="0.1524" layer="91"/>
 <pinref part="U1" gate="A" pin="OUT"/>
 <wire x1="71.12" y1="220.98" x2="73.66" y2="220.98" width="0.1524" layer="91"/>
-<wire x1="73.66" y1="220.98" x2="73.66" y2="208.28" width="0.1524" layer="91"/>
-<junction x="73.66" y="208.28"/>
+<wire x1="73.66" y1="220.98" x2="73.66" y2="213.614" width="0.1524" layer="91"/>
 <pinref part="+3V1" gate="G$1" pin="+3V3"/>
 <wire x1="73.66" y1="220.98" x2="86.36" y2="220.98" width="0.1524" layer="91"/>

Commit message: Added version 1.0
Parts:
- removed H1, H2, H3, H4: MOUNTINGHOLE2.5, milador:MOUNTINGHOLE2.5
- removed J1: JACDAC_EDGE_CONN-INNIE, Jacdac:JACDAC_EDGE_CONN-INNIE
- removed LABEL2: JACDAC-DEVICE-PS, milador:JACDAC-DEVICE-PS
- removed U$1: JACDAC-DEVICE-LPS33HW, milador:JACDAC-DEVICE-LPS33HW
- added J3: 5V, milador:JACDAC-M3-PWR-OUTL
- added J4: DATA, milador:JACDAC-M3-DATA-NOTCH
- added J5, J6: GND, milador:JACDAC-M3-GND
- added JD1, JD2: JACDAC-EDGE-OUTIE, milador:JACDAC-EDGE-OUTIE
- added LABEL_JACDAC_PS: MILADOR-JACDAC-DEVICE-PS, milador:MILADOR-JACDAC-DEVICE-PS
- added LABEL_LPS33HW: MILADOR-JACDAC-DEVICE-LPS33HW, milador:MILADOR-JACDAC-DEVICE-LPS33HW
- added LABEL_QR_CODE: MILADOR-QR-CODE-JACDAC-GITHUB-PS, milador:MILADOR-QR-CODE-JACDAC-GITHUB-PS
- C1: value 0.1uF -> 1uF
- C2: value 1uF -> 33pF; device milador_SMD:CAP_CERAMIC-0603-NO -> milador_SMD:CAP_CERAMIC-0603
- C3: value 33pF -> 1uF; device milador_SMD:CAP_CERAMIC-0603 -> milador_SMD:CAP_CERAMIC-0603-NO
- C4: value 1uF -> 0.1uF
- D1: value LED-HSMF-C114 -> DIODE-ZENER-AA-RCLAMP0521PATCT; device milador_SMD:LED-HSMF-C114 -> milador_SMD:DIODE-ZENER-AA-RCLAMP0521PATCT
- D2: value RCLAMP0521PATCT -> DIODE-ZENER-AA-RCLAMP0521PATCT; device milador_SMD:DIODE-ZENER-RCLAMP0521PATCT -> milador_SMD:DIODE-ZENER-AA-RCLAMP0521PATCT
- D3: value RCLAMP0521PATCT -> LED-HSMF-C114; device milador_SMD:DIODE-ZENER-RCLAMP0521PATCT -> milador_SMD:LED-HSMF-C114
- MMC_LOGO: value MMC_LOGO-SM -> MMC_LOGO-XSM; device MMC Eagle:MMC_LOGO-SM -> MMC Eagle:MMC_LOGO-XSM
- U1: value NCP114ASN330T1G -> STM32F042F6P6; device milador_SMD:NCP114ASN330T1G -> milador_SMD:STM32F042F6P6
- U2: value STM32F042F6P6 -> NCP114ASN330T1G; device milador_SMD:STM32F042F6P6 -> milador_SMD:NCP114ASN330T1G
- renumbered LABEL3 to LABEL_MILADOR
Connections:
- net +3V3: now also C3.1, D3.1, U1.VDD, U1.VDDA, U2.OUT; no longer C1.1, D1.1, U1.OUT, U2.VDD, U2.VDDA
- net GND: now also D1.A, J5.P$1, J6.P$1, JD1.1, JD2.1, U1.BOOT0, U1.VSS, U2.GND; no longer D3.A, H3.P$1, H4.P$1, J1.2, U1.GND, U2.BOOT0, U2.VSS
- net JD_DATA: now also U1.PA2; no longer U2.PA2
- net J_DATA: now also D2.A2, J4.P$1, JD1.2, JD1.6, JD2.2, JD2.6; no longer D3.A2, H2.P$1, J1.1
- net N$1: now also D3.4; no longer D1.4
- net N$2: now also D3.3; no longer D1.3
- net N$3: now also D3.2; no longer D1.2
- net N$4: now also C2.1; no longer C3.1
- net RESET: now also U1.!RST; no longer U2.!RST
- net RGB_B: now also U1.PB1; no longer U2.PB1
- net RGB_G: now also U1.PA4; no longer U2.PA3
- net RGB_R: now also U1.PA3; no longer U2.PA4
- net SCL: now also U1.PA11; no longer U2.PA11
- net SDA: now also U1.PA12; no longer U2.PA12
- net SWCLK: now also U1.PA14; no longer U2.PA14
- net SWDIO: now also U1.PA13; no longer U2.PA13
- net VCC: now also C1.1, D1.A2, J3.P$1, JD1.3, JD1.4, JD2.3, JD2.4, U2.EN, U2.IN; no longer C2.1, D2.A2, H1.P$1, J1.3, U1.EN, U1.IN
Other:
- note added: "Jacdac Connector 2"
- note added: "STM32F042F6P6"
- note removed: "MakersMakingChange"
- moved on the sheet: C1, C2, C3, C4, D2, FB1, R4, U4
