File: Hardware/PCB/Eagle/Jacdac_Pressure_Sensor-RevA-Maker.sch (EAGLE design)
At the start: 29 parts, among them J2 SWD-ADAPTER-, J3 5V, J4 DATA, J5 GND, J6 GND, U1 STM32F042F6P6, U2 NCP114ASN330T1G, U3 LPS33HWTR, U4 BAT54S,235

Commit message: Updated revision A
Connections:
- net +3V3: now also U3.CS
Changed lines of the file:
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@@
 <part name="GND14" library="SparkFun-PowerSymbols" deviceset="GND" device=""/>
 <part name="LABEL_QR_CODE" library="milador" library_urn="urn:adsk.eagle:library:12595918" deviceset="MILADOR-QR-CODE-" device="JACDAC-GITHUB-PS" package3d_urn="urn:adsk.eagle:package:36433227/1"/>
+<part name="+3V7" library="supply1" library_urn="urn:adsk.eagle:library:371" deviceset="+3V3" device=""/>
 </parts>
 <sheets>
@@
 </instance>
 <instance part="LABEL_QR_CODE" gate="G$1" x="312.42" y="75.438" smashed="yes"/>
+<instance part="+3V7" gate="G$1" x="13.208" y="60.452" smashed="yes">
+<attribute name="VALUE" x="10.668" y="55.372" size="1.778" layer="96" rot="R90"/>
+</instance>
 </instances>
 <busses>
@@
 <wire x1="88.9" y1="47.752" x2="88.9" y2="63.292" width="0.1524" layer="91"/>
 </segment>
+<segment>
+<pinref part="U3" gate="G$1" pin="CS"/>
+<pinref part="+3V7" gate="G$1" pin="+3V3"/>
+<wire x1="20.574" y1="50.038" x2="13.208" y2="50.038" width="0.1524" layer="91"/>
+<wire x1="13.208" y1="50.038" x2="13.208" y2="57.912" width="0.1524" layer="91"/>
+</segment>
 </net>
