File: Hardware/PCB/Eagle/Jacdac_Pressure_Sensor-RevA.brd (EAGLE design)
At the start: 25 x 25 mm, 31 parts, among them J2 SWD-ADAPTER-, J3 5V, J4 DATA, J5 GND, J6 GND, U1 STM32F042F6P6, U2 NCP114ASN330T1G, U3 LPS33HWTR, U4 BAT54S,235

Commit message: Updated revision A
Connections:
- net +3V3: now also U3.6
Routing:
- net +3V3: track 47.4 -> 54.6 mm
Changed lines of the file:
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@@
 </layers>
 <board>
-<fusionsync huburn="a.cGVyc29uYWw6dWUyYWQxOTI2" projecturn="a.cGVyc29uYWw6dWUyYWQxOTI2IzIwMjEwOTEzNDQzNTc2ODA2" f3durn="urn:adsk.wipprod:dm.lineage:vh679-O6RLKkiJJlloXqaw" pcbguid="" lastpulledtime="" lastsyncedchangeguid="" latestrevisionid="d66f17c6-5d52-4ebd-afb4-393af988ddbe" lastsyncedrevisionid="d66f17c6-5d52-4ebd-afb4-393af988ddbe" lastboardhashguid="4326f1c8-6fc1-c811-7cf0-6b2e3d2b8987" lastpushedtime="2022-07-09T01:37:09Z" linktopcb3d="true"/>
+<fusionsync huburn="a.cGVyc29uYWw6dWUyYWQxOTI2" projecturn="a.cGVyc29uYWw6dWUyYWQxOTI2IzIwMjEwOTEzNDQzNTc2ODA2" f3durn="urn:adsk.wipprod:dm.lineage:vh679-O6RLKkiJJlloXqaw" pcbguid="" lastpulledtime="" lastsyncedchangeguid="" latestrevisionid="d66f17c6-5d52-4ebd-afb4-393af988ddbe" lastsyncedrevisionid="d66f17c6-5d52-4ebd-afb4-393af988ddbe" lastboardhashguid="4326f1c8-6fc1-c811-7cf0-6b2e3d2b8987" lastpushedtime="2022-07-09T01:37:09Z" linktopcb3d="false"/>
 <plain>
 <wire x1="4" y1="25" x2="6" y2="25" width="0.05" layer="20"/>
@@
 <wire x1="8.55" y1="13.83308125" x2="8.455" y2="13.92808125" width="0.2" layer="1"/>
 <wire x1="8.55" y1="13.83308125" x2="8.55" y2="12.33985" width="0.2" layer="1"/>
-<wire x1="19.35" y1="17.607003125" x2="19.35" y2="17.25" width="0.2" layer="1"/>
-<wire x1="19.35" y1="17.607003125" x2="17.65" y2="19.307003125" width="0.2" layer="1"/>
-<wire x1="17.65" y1="19.5" x2="17.65" y2="19.307003125" width="0.2" layer="1"/>
 <wire x1="19.6" y1="14.5" x2="19.6" y2="14.098359375" width="0.2" layer="1"/>
 <wire x1="17.815559375" y1="12.31391875" x2="17.815559375" y2="11.5" width="0.2" layer="1"/>
@@
 <wire x1="13.07591875" y1="6.2" x2="13.07591875" y2="1.83311875" width="0.2" layer="1"/>
 <wire x1="13.07591875" y1="1.83311875" x2="13.075" y2="1.8322" width="0.2" layer="1"/>
+<contactref element="U3" pad="6"/>
+<wire x1="14.3" y1="13.82" x2="14.95791875" y2="13.82" width="0.2" layer="1"/>
+<wire x1="14.95791875" y1="13.82" x2="15.585440625" y2="14.447521875" width="0.2" layer="1"/>
+<wire x1="15.585440625" y1="14.447521875" x2="15.585440625" y2="16.8249625" width="0.2" layer="1"/>
+<wire x1="15.585440625" y1="16.8249625" x2="17.170396875" y2="18.40991875" width="0.2" layer="1"/>
+<wire x1="17.170396875" y1="18.40991875" x2="17.64791875" y2="18.40991875" width="0.2" layer="1"/>
+<wire x1="17.64791875" y1="18.40991875" x2="18.63344375" y2="18.40991875" width="0.2" layer="1"/>
+<wire x1="17.65" y1="19.5" x2="17.65" y2="18.412" width="0.2" layer="1"/>
+<wire x1="17.65" y1="18.412" x2="17.64791875" y2="18.40991875" width="0.2" layer="1"/>
+<wire x1="18.63344375" y1="18.40991875" x2="19.35" y2="17.6933625" width="0.2" layer="1"/>
+<wire x1="19.35" y1="17.6933625" x2="19.35" y2="17.25" width="0.2" layer="1"/>
 </signal>
 <signal name="RESET">
