File: Hardware/PCB/Eagle/Jacdac_Pressure_Sensor-RevA.sch (EAGLE design)
At the start: 31 parts, among them J2 SWD-ADAPTER-, J3 5V, J4 DATA, J5 GND, J6 GND, U1 STM32F042F6P6, U2 NCP114ASN330T1G, U3 LPS33HWTR, U4 BAT54S,235

Commit message: Updated revision A
Connections:
- net +3V3: now also U3.CS
Changed lines of the file:
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@@
 <part name="D2" library="milador_SMD" library_urn="urn:adsk.eagle:library:27847482" deviceset="DIODE-ZENER-AA-" device="RCLAMP0521PATCT" package3d_urn="urn:adsk.eagle:package:30689290/6"/>
 <part name="LABEL_QR_CODE" library="milador" library_urn="urn:adsk.eagle:library:12595918" deviceset="MILADOR-QR-CODE-" device="JACDAC-GITHUB-PS" package3d_urn="urn:adsk.eagle:package:36433227/1"/>
+<part name="+3V7" library="supply1" library_urn="urn:adsk.eagle:library:371" deviceset="+3V3" device=""/>
 </parts>
 <sheets>
@@
 </instance>
 <instance part="LABEL_QR_CODE" gate="G$1" x="312.42" y="75.438" smashed="yes"/>
+<instance part="+3V7" gate="G$1" x="12.192" y="60.198" smashed="yes">
+<attribute name="VALUE" x="9.652" y="55.118" size="1.778" layer="96" rot="R90"/>
+</instance>
 </instances>
 <busses>
@@
 <wire x1="88.9" y1="47.752" x2="88.9" y2="63.292" width="0.1524" layer="91"/>
 </segment>
+<segment>
+<pinref part="U3" gate="G$1" pin="CS"/>
+<pinref part="+3V7" gate="G$1" pin="+3V3"/>
+<wire x1="20.574" y1="50.038" x2="12.192" y2="50.038" width="0.1524" layer="91"/>
+<wire x1="12.192" y1="50.038" x2="12.192" y2="57.658" width="0.1524" layer="91"/>
+</segment>
 </net>
